Commit message: where am I

File: my_robot/urdf/my_robot.xacro (robot description, xacro)
@@ -1,5 +1,6 @@
+<?xml version='1.0'?>
 <robot name="my_robot" xmlns:xacro="http://www.ros.org/wiki/xacro">
+    <xacro:include filename="/home/robond/catkin_ws/src/my_robot/urdf/my_robot.gazebo" />
     <link name="robot_footprint"></link>
-    <xacro:include filename="$(find my_robot)/urdf/my_robot.gazebo" />
     <joint name="robot_footprint_joint" type="fixed">
         <origin xyz="0 0 0" rpy="0 0 0" />
@@ -7,13 +8,4 @@
         <child link="chassis" />
     </joint>
-    <gazebo reference="chassis">
-        <material>Gazebo/Orange</material>
-    </gazebo>
-    <gazebo reference="left_wheel">
-        <material>Gazebo/Black</material>
-    </gazebo>
-    <gazebo reference="right_wheel">
-        <material>Gazebo/Black</material>
-    </gazebo>
     <link name='chassis'>
         <pose>0 0 0.1 0 0 0</pose>
@@ -89,4 +81,12 @@
         </collision>
     </link>
+    <joint name="left_wheel_hinge" type="continuous">
+        <origin xyz="0.0 0.15 0.0" rpy="0.0 0.0 0.0"/>
+        <parent link="chassis"/>
+        <child link="left_wheel"/>
+        <axis xyz="0.0 1.0 0.0" rpy="0.0 0.0 0.0"/>
+        <limit lower="0.0" upper="0.0" effort="1000.0" velocity="1000.0"/>
+        <dynamics damping="1.0" friction="1.0"/>
+    </joint>
     <link name="right_wheel">
         <pose>0.0 0.0 0.1 0 0 0</pose>
@@ -114,4 +114,37 @@
         </collision>
     </link>
+    <joint name="right_wheel_hinge" type="continuous">
+        <origin xyz="0.0 -0.15 0.0" rpy="0.0 0.0 0.0"/>
+        <parent link="chassis"/>
+        <child link="right_wheel"/>
+        <axis xyz="0.0 1.0 0.0" rpy="0.0 0.0 0.0"/>
+        <limit lower="0.0" upper="0.0" effort="1000.0" velocity="1000.0"/>
+        <dynamics damping="1.0" friction="1.0"/>
+    </joint>
+    <link name="hokuyo">
+        <inertial>
+            <mass value="1e-5"/>
+            <origin xyz="0.0 0.0 0.0" rpy="0.0 0.0 0.0"/>
+            <inertia ixx="1e-6" ixy="0.0" ixz="0.0" iyy="1e-6" iyz="0.0" izz="1e-6"/>
+        </inertial>
+        <visual>
+            <origin xyz="0.0 0.0 0.0" rpy="0.0 0.0 0.0"/>
+            <geometry>
+                <mesh filename="package://my_robot/meshes/hokuyo.dae"/>
+            </geometry>
+        </visual>
+        <collision>
+            <origin xyz="0.0 0.0 0.0" rpy="0.0 0.0 0.0"/>
+            <geometry>
+                <box size="0.1 0.1 0.1"/>
+            </geometry>
+        </collision>
+    </link>
+    <joint name="hokuyo_joint" type="fixed">
+        <origin xyz="0.15 0.0 0.1" rpy="0.0 0.0 0.0"/>
+        <axis xyz="0.0 1.0 0.0"/>
+        <parent link="chassis"/>
+        <child link="hokuyo"/>
+    </joint>
     <link name="camera">
         <inertial>
@@ -133,48 +166,4 @@
         </collision>
     </link>
-    <link name="hokuyo">
-        <inertial>
-            <mass value="1e-5"/>
-            <origin xyz="0.0 0.0 0.0" rpy="0.0 0.0 0.0"/>
-            <inertia ixx="1e-6" ixy="0.0" ixz="0.0" iyy="1e-6" iyz="0.0" izz="1e-6"/>
-        </inertial>
-        <visual>
-            <origin xyz="0.0 0.0 0.0" rpy="0.0 0.0 0.0"/>
-            <geometry>
-                <mesh filename="package://my_robot/meshes/hokuyo.dae"/>
-            </geometry>
-        </visual>
-        <collision>
-            <origin xyz="0.0 0.0 0.0" rpy="0.0 0.0 0.0"/>
-            <geometry>
-                <box size="0.1 0.1 0.1"/>
-            </geometry>
-        </collision>
-    </link>
-    <gazebo reference="camera">
-        <material>Gazebo/Grey</material>
-    </gazebo>
-    <joint name="left_wheel_hinge" type="continuous">
-        <origin xyz="0.0 0.15 0.0" rpy="0.0 0.0 0.0"/>
-        <parent link="chassis"/>
-        <child link="left_wheel"/>
-        <axis xyz="0.0 1.0 0.0" rpy="0.0 0.0 0.0"/>
-        <limit lower="0.0" upper="0.0" effort="1000.0" velocity="1000.0"/>
-        <dynamics damping="1.0" friction="1.0"/>
-    </joint>
-    <joint name="right_wheel_hinge" type="continuous">
-        <origin xyz="0.0 -0.15 0.0" rpy="0.0 0.0 0.0"/>
-        <parent link="chassis"/>
-        <child link="right_wheel"/>
-        <axis xyz="0.0 1.0 0.0" rpy="0.0 0.0 0.0"/>
-        <limit lower="0.0" upper="0.0" effort="1000.0" velocity="1000.0"/>
-        <dynamics damping="1.0" friction="1.0"/>
-    </joint>
-    <joint name="hokuyo_joint" type="fixed">
-        <origin xyz="0.15 0.0 0.1" rpy="0.0 0.0 0.0"/>
-        <axis xyz="0.0 1.0 0.0"/>
-        <parent link="chassis"/>
-        <child link="hokuyo"/>
-    </joint>
     <joint name="camera_joint" type="fixed">
         <origin xyz="0.2 0.0 0.0" rpy="0.0 0.0 0.0"/>
@@ -183,3 +172,15 @@
         <child link="camera"/>
     </joint>
+    <gazebo reference="camera">
+        <material>Gazebo/Grey</material>
+    </gazebo>
+    <gazebo reference="chassis">
+        <material>Gazebo/Orange</material>
+    </gazebo>
+    <gazebo reference="left_wheel">
+        <material>Gazebo/Black</material>
+    </gazebo>
+    <gazebo reference="right_wheel">
+        <material>Gazebo/Black</material>
+    </gazebo>
 </robot>

Commit message: slam_changes

File: my_robot/urdf/my_robot.xacro (robot description, xacro)
@@ -142,5 +142,5 @@
     </link>
     <joint name="hokuyo_joint" type="fixed">
-        <origin xyz="0.15 0.0 0.1" rpy="0.0 0.0 0.0"/>
+        <origin xyz="0.15 0.0 0.15  " rpy="0.0 0.0 0.0"/>
         <axis xyz="0.0 1.0 0.0"/>
         <parent link="chassis"/>
@@ -154,5 +154,5 @@
         </inertial>
         <visual>
-            <origin xyz="0.2 0.0 0.0" rpy="0.0 0.0 0.0"/>
+            <origin xyz="0.0 0.0 0.0" rpy="0.0 0.0 0.0"/>
             <geometry>
                 <box size="0.05 0.05 0.05"/>
@@ -160,5 +160,5 @@
         </visual>
         <collision>
-            <origin xyz="0.2 0.0 0.0" rpy="0.0 0.0 0.0"/>
+            <origin xyz="0.0 0.0 0.0" rpy="0.0 0.0 0.0"/>
             <geometry>
                 <box size="0.05 0.05 0.05"/>
@@ -175,4 +175,11 @@
         <material>Gazebo/Grey</material>
     </gazebo>
+    <joint name="camera_optical_joint" type="fixed">
+        <origin xyz="0.0 0.0 0.0" rpy="-1.5707 0.0 -1.5707"/>
+        <parent link="camera"/>
+        <child link="camera_link_optical"/>
+    </joint>
+    <link name="camera_link_optical">
+    </link>
     <gazebo reference="chassis">
         <material>Gazebo/Orange</material>
